File: mainboard-ng.kicad_sch (KiCad schematic)
At the start: 0 parts

Commit message: done
Parts:
- added C16, C17: 0.1uF, Capacitor_SMD:C_0805_2012Metric_Pad1.18x1.45mm_HandSolder, symbol Device:C
- added J1, J2: Conn_01x15_Socket, Connector_PinSocket_2.54mm:PinSocket_1x15_P2.54mm_Vertical, symbol Connector:Conn_01x15_Socket
- added J3: Sensor, Connector_PinHeader_2.54mm:PinHeader_1x11_P2.54mm_Vertical, symbol Connector:Conn_01x11_Pin
- added J4: Conn_01x02_Pin, Connector_PinSocket_2.54mm:PinSocket_1x02_P2.54mm_Vertical, symbol Connector:Conn_01x02_Pin
- added PWR1: (no value), #lineracer:PWR, symbol #lineracer:Powermodule
- added R1: 100k, Resistor_THT:R_Axial_DIN0309_L9.0mm_D3.2mm_P5.08mm_Vertical, symbol Device:R
- added R2: 20K, Resistor_THT:R_Axial_DIN0309_L9.0mm_D3.2mm_P5.08mm_Vertical, symbol Device:R
- added R4: 1.8k, Resistor_THT:R_Axial_DIN0309_L9.0mm_D3.2mm_P5.08mm_Vertical, symbol Device:R
- added R5: 3.3k, Resistor_THT:R_Axial_DIN0309_L9.0mm_D3.2mm_P5.08mm_Vertical, symbol Device:R
- added U1: (no value), ESP32_Footprints:ESP32_30pin_mod, symbol esp32_30pin_revised:ESP32_30Pin
- added U3: MCP3208, Package_DIP:DIP-16_W7.62mm_LongPads, symbol Analog_ADC:MCP3208
- added U4: SN74AHCT125DR, Package_DIP:DIP-14_W10.16mm_LongPads, symbol SN74AHCT125DR:SN74AHCT125DR
Connections:
- new net: J3.2 (Pin_2), U3.1 (CH0)
- new net: U3.10 (~{CS}/SHDN), U4.6 (2Y)
- new net: U3.11 (Din), U4.8 (3Y)
- new net: R4.1, U3.12 (Dout)
- new net: U3.13 (CLK), U4.11 (4Y)
- new net: J3.3 (Pin_3), U3.2 (CH1)
- new net: J3.4 (Pin_4), U3.3 (CH2)
- new net: J3.5 (Pin_5), U3.4 (CH3)
- new net: J3.6 (Pin_6), U3.5 (CH4)
- new net: J3.7 (Pin_7), U3.6 (CH5)
- new net: J3.8 (Pin_8), U3.7 (CH6)
- new net: J3.9 (Pin_9), U3.8 (CH7)
- new net: J3.10 (Pin_10), U4.3 (1Y)
- new net: J1.12 (Pin_12), U1.12 (GPIO34)
- new net: J1.13 (Pin_13), U1.13 (GPIO39)
- new net: J1.15 (Pin_15), U1.15 (EN)
- new net: J2.15 (Pin_15), U1.16 (3.3v)
- new net: J2.13 (Pin_13), U1.18 (GPIO15)
- new net: J2.12 (Pin_12), U1.19 (GPIO2)
- new net: J1.2 (Pin_2), U1.2 (GND)
- new net: J2.10 (Pin_10), U1.21 (GPIO16)
- new net: J2.9 (Pin_9), U1.22 (GPIO17)
- new net: J2.8 (Pin_8), U1.23 (GPIO5)
- new net: J2.7 (Pin_7), U1.24 (GPIO18)
- new net: J2.6 (Pin_6), U1.25 (GPIO19)
- new net: J2.5 (Pin_5), U1.26 (GPIO21)
- new net: J2.4 (Pin_4), U1.27 (GPIO3)
- new net: J2.3 (Pin_3), U1.28 (GPIO1)
- new net: J2.2 (Pin_2), U1.29 (GPIO22)
- new net: J2.1 (Pin_1), U1.30 (GPIO23)
- new net: J1.4 (Pin_4), U1.4 (GPIO12)
- new net: J1.6 (Pin_6), U1.6 (GPIO27)
- new net: J1.7 (Pin_7), U1.7 (GPIO26)
- new net: J1.8 (Pin_8), U1.8 (GPIO25)
- new net: J1.9 (Pin_9), U1.9 (GPIO33)
- new net +5V: C16.1, C17.1, J1.1 (Pin_1), J3.11 (Pin_11), PWR1.4 (VOUT), U1.1 (VIN), U3.15 (Vref), U3.16 (Vdd), U4.14 (VCC)
- new net BATMON: J1.14 (Pin_14), R1.2, R2.1, U1.14 (GPIO36)
- new net BATPWR: J4.1 (Pin_1), PWR1.2 (VIN), R1.1
- new net CLK: J1.5 (Pin_5), U1.5 (GPIO14), U4.12 (4A)
- new net CS: J2.11 (Pin_11), U1.20 (GPIO4), U4.5 (2A)
- new net GND: C16.2, C17.2, J2.14 (Pin_14), J3.1 (Pin_1), J4.2 (Pin_2), PWR1.3 (GND), R2.2, R5.2, U1.17 (GND), U3.14 (AGND), U3.9 (DGND), U4.1 (1~{OE}), U4.10 (3~{OE}), U4.13 (4~{OE}), U4.4 (2~{OE}), U4.7 (GND)
- new net IR: J1.10 (Pin_10), U1.10 (GPIO32), U4.2 (1A)
- new net MISO: J1.11 (Pin_11), R4.2, R5.1, U1.11 (GPIO35)
- new net MOSI: J1.3 (Pin_3), U1.3 (GPIO13), U4.9 (3A)
