File: mainboard.ng/mainboard-ng.kicad_pcb (KiCad board)
At the start: 2 copper layers, 40 x 60 mm, 16 parts, among them J1 Conn_01x15_Socket, J2 Conn_01x15_Socket, J3 Sensor, J4 Conn_01x02_Pin, U3 MCP3208, U4 SN74AHCT125DR

Commit message: move to subfolder
Parts:
- renumbered REF** to REF1, REF** to REF2
Changed lines of the file:
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@@
 	)
 	(paper "A4")
+	(title_block
+		(comment 4 "AISLER Project ID: RBBPVEFK")
+	)
 	(layers
 		(0 "F.Cu" signal)
@@
 			(plotframeref no)
 			(mode 1)
-			(useauxorigin no)
+			(useauxorigin yes)
 			(pdf_front_fp_property_popups yes)
 			(pdf_back_fp_property_popups yes)
@@
 			(outputformat 1)
 			(mirror no)
-			(drillshape 1)
+			(drillshape 0)
 			(scaleselection 1)
-			(outputdirectory "")
+			(outputdirectory "manufacturing-export")
 		)
 	)
@@
 		(descr "Mounting Hole 2.2mm, M2, generated by kicad-footprint-generator mountinghole.py")
 		(tags "mountinghole M2 DIN965")
-		(property "Reference" "REF**"
+		(property "Reference" "REF2"
 			(at 0 -2.85 0)
 			(layer "F.SilkS")
@@
 		(descr "Mounting Hole 2.2mm, M2, generated by kicad-footprint-generator mountinghole.py")
 		(tags "mountinghole M2 DIN965")
-		(property "Reference" "REF**"
+		(property "Reference" "REF1"
 			(at 0 -2.85 0)
 			(layer "F.SilkS")
